Commit message: Add SAC and CV modules, remove large files

File: install/robot_gazebo/share/robot_gazebo/urdf/camera.gazebo.xacro (robot description, xacro)
@@ -1 +1,24 @@
-/workspaces/ros2_ws/build/robot_gazebo/urdf/camera.gazebo.xacro
+<?xml version="1.0" encoding="utf-8" ?>
+<robot name="camera_gazebo" xmlns:xacro="http://ros.org/wiki/xacro">
+  <gazebo reference="camera_link0">
+    <sensor name="robot_cam" type="camera">
+      <camera>
+        <horizontal_fov>1.047</horizontal_fov>
+        <image>
+          <width>640</width>
+          <height>400</height>
+        </image>
+        <clip>
+          <near>0.1</near>
+          <far>10</far>
+        </clip>
+      </camera>
+      <always_on>1</always_on>
+      <update_rate>30</update_rate>
+      <visualize>true</visualize>
+      <camera_info_topic>/depth_cam/rgb/camera_info</camera_info_topic>
+      <topic>/depth_cam/depth_cam</topic>
+      <enable_metrics>true</enable_metrics>
+    </sensor>
+  </gazebo>
+</robot>

File: install/robot_gazebo/share/robot_gazebo/urdf/imu.gazebo.xacro (robot description, xacro)
@@ -1 +1,12 @@
-/workspaces/ros2_ws/build/robot_gazebo/urdf/imu.gazebo.xacro
+<?xml version="1.0" encoding="utf-8" ?>
+<robot xmlns:xacro="http://www.ros.org/wiki/xacro" name="robot_imu">
+    <gazebo reference="imu_link">
+        <sensor name="imu_sensor" type="imu">
+            <always_on>1</always_on>
+            <update_rate>50</update_rate>
+            <ignition_frame_id>imu_link</ignition_frame_id>
+            <visualize>true</visualize>
+            <topic>imu</topic>
+        </sensor>
+    </gazebo>
+</robot>

File: install/robot_gazebo/share/robot_gazebo/urdf/lidar.gazebo.xacro (robot description, xacro)
@@ -1 +1,33 @@
-/workspaces/ros2_ws/build/robot_gazebo/urdf/lidar.gazebo.xacro
+<?xml version="1.0"?>
+<robot xmlns:xacro="http://www.ros.org/wiki/xacro" name="gpu_lidar">
+    <gazebo reference="lidar_frame">
+        <sensor name="gpu_lidar" type="gpu_lidar">
+            <!-- <pose>0 0 0 0 0 0</pose>             -->
+            <topic>scan</topic>
+            <update_rate>10</update_rate>
+            <ignition_frame_id>lidar_frame</ignition_frame_id>
+            <ray>
+                <scan>
+                    <horizontal>
+                        <samples>270</samples>
+                        <resolution>1</resolution>
+                        <min_angle>-1.36263</min_angle>
+                        <max_angle>1.36263</max_angle>
+                    </horizontal>
+                </scan>
+                <range>
+                    <min>0.15</min>
+                    <max>12.0</max>
+                    <resolution>0.01</resolution>
+                </range>
+                <noise>
+                    <type>gaussian</type>
+                    <mean>0.0</mean>
+                    <stddev>0.01</stddev>
+                </noise>
+            </ray>
+            <alwaysOn>1</alwaysOn>
+            <visualize>true</visualize>
+        </sensor>
+    </gazebo>
+</robot>

File: install/robot_gazebo/share/robot_gazebo/urdf/robot.gazebo.xacro (robot description, xacro)
@@ -1 +1,61 @@
-/workspaces/ros2_ws/build/robot_gazebo/urdf/robot.gazebo.xacro
+<?xml version="1.0" encoding="utf-8"?>
+<robot name="robot" xmlns:xacro="http://ros.org/wiki/xacro">
+    <xacro:arg name="sim_ign" default="true"/>
+    <!-- robot_description -->
+    <xacro:include filename="$(find rosorin_description)/urdf/rosorin.xacro"/>
+    <xacro:if value="$(arg sim_ign)">
+        <xacro:include filename="$(find robot_gazebo)/urdf/wheel.xacro"/>
+    </xacro:if>
+    <!-- lidar -->
+    <xacro:include filename="$(find robot_gazebo)/urdf/lidar.gazebo.xacro"/>
+    <!-- camera -->
+    <xacro:include filename="$(find robot_gazebo)/urdf/camera.gazebo.xacro"/>
+    <gazebo>
+        <!-- Joint state publisher -->
+        <plugin filename="$(find ign_ros2_control)/../../lib/libign_ros2_control-system.so"
+                name="ign_ros2_control::IgnitionROS2ControlPlugin">
+          <parameters>$(find robot_gazebo)/config/robot_config.yaml</parameters>
+        </plugin>
+        <!-- joint -->
+        <plugin filename="libignition-gazebo-joint-state-publisher-system.so" name="ignition::gazebo::systems::JointStatePublisher">
+            <topic>joint_states</topic>
+        </plugin>
+        <!-- sensor-liar -->
+        <plugin filename="ignition-gazebo-sensors-system" name="ignition::gazebo::systems::Sensors">
+            <render_engine>ogre2</render_engine>
+        </plugin>
+        <!-- imu -->
+        <plugin filename="ignition-gazebo-imu-system" name="ignition::gazebo::systems::Imu"></plugin>
+        <!-- odom -->
+        <plugin
+            filename="ignition-gazebo-odometry-publisher-system"
+            name="ignition::gazebo::systems::OdometryPublisher">
+            <odom_publish_frequency>50</odom_publish_frequency>
+            <odom_topic>/odom</odom_topic>
+            <odom_frame>odom</odom_frame>
+            <robot_base_frame>base_footprint</robot_base_frame>
+            <tf_topic>/odom/tf</tf_topic>
+        </plugin>
+        <!-- Holonomic plugin -->
+        <!-- <xacro:if value="$(arg sim_ign)">
+            <plugin filename="libHolonomicPlugin.so" name="holonomic_sim::HolonomicPlugin">
+                <wheel_joint>wheel_joint</wheel_joint>
+                <top_base_joint>top_wheel_base_joint</top_base_joint>
+                <bottom_base_joint>bottom_wheel_base_joint</bottom_base_joint>
+            </plugin>
+        </xacro:if> -->
+    <plugin filename="ignition-gazebo-mecanum-drive-system" name="ignition::gazebo::systems::MecanumDrive">
+        <front_left_joint>front_left_joint</front_left_joint>
+        <front_right_joint>front_right_joint</front_right_joint>
+        <back_left_joint>rear_left_joint</back_left_joint>
+        <back_right_joint>rear_right_joint</back_right_joint>
+        <wheel_separation>0.34</wheel_separation>
+        <wheelbase>0.3</wheelbase>
+        <wheel_radius>0.05</wheel_radius>
+	<topic>/controller/cmd_vel</topic>
+        <odom_topic>/odom</odom_topic>
+        <frame_id>odom</frame_id>
+        <child_frame_id>base_link</child_frame_id>
+        </plugin>
+    </gazebo>
+</robot>

File: install/robot_gazebo/share/robot_gazebo/urdf/wheel.xacro (robot description, xacro)
@@ -1 +1,46 @@
-/workspaces/ros2_ws/build/robot_gazebo/urdf/wheel.xacro
+<?xml version="1.0"?>
+<robot xmlns:xacro="http://www.ros.org/wiki/xacro">
+  <!-- ============================================== -->
+  <xacro:property name="WHEEL_RADIUS" value="0.04" />
+  <xacro:property name="WHEEL_LENGTH" value="0.025" />
+  <xacro:property name="WHEEL_VISUAL_ENABLE" value="true" />
+  <!-- ============================================== -->
+  <xacro:macro name="mecanum_wheel" params="name x y">
+    <link name="${name}_link">
+      <xacro:if value="${WHEEL_VISUAL_ENABLE}">
+        <visual>
+          <geometry><cylinder radius="${WHEEL_RADIUS}" length="${WHEEL_LENGTH}"/></geometry>
+          <material name="black"><color rgba="0 0 0 1"/></material>
+          <origin rpy="1.5707 0 0"/>
+        </visual>
+      </xacro:if>
+      <collision>
+        <geometry><cylinder radius="${WHEEL_RADIUS}" length="${WHEEL_LENGTH}"/></geometry>
+        <origin rpy="1.5707 0 0"/>
+      </collision>
+      <inertial>
+        <mass value="10.0"/>
+        <inertia ixx="0.0007" ixy="0" ixz="0" iyy="0.0007" iyz="0" izz="0.0012"/>
+      </inertial>
+    </link>
+    <joint name="${name}_joint" type="continuous">
+      <parent link="base_link"/>
+      <child link="${name}_link"/>
+      <origin xyz="${x} ${y} 0.01"/>
+      <axis xyz="0 1 0"/>
+      <dynamics damping="1.0" friction="0.5"/>
+    </joint>
+    <gazebo reference="${name}_link">
+      <mu1>10.0</mu1>
+      <mu2>10.0</mu2>
+      <kp>1000000000.0.0</kp>
+      <kd>100000.0</kd>
+      <minDepth>0.0001</minDepth>
+    </gazebo>
+  </xacro:macro>
+  <!-- ============================================== -->
+  <xacro:mecanum_wheel name="front_left"  x="0.08"  y="0.09"/>
+  <xacro:mecanum_wheel name="front_right" x="0.08"  y="-0.09"/>
+  <xacro:mecanum_wheel name="rear_left"   x="-0.08" y="0.09"/>
+  <xacro:mecanum_wheel name="rear_right"  x="-0.08" y="-0.09"/>
+</robot>

File: install/rosorin_description/share/rosorin_description/urdf/ascamera.xacro (robot description, xacro)
@@ -1 +1,56 @@
-/workspaces/ros2_ws/build/rosorin_description/urdf/ascamera.xacro
+<?xml version="1.0" encoding="utf-8"?>
+<robot name="camera" xmlns:xacro="http://ros.org/wiki/xacro" >
+  <link
+    name="camera_link0">
+    <inertial>
+      <origin
+        xyz="0.00232997875786055 -0.000556155071961858 -2.82983961463062E-05"
+        rpy="0 0 0" />
+      <mass
+        value="0.015428346878935" />
+      <inertia
+        ixx="1.36095493821731E-05"
+        ixy="2.31032732804664E-07"
+        ixz="-1.31690079926083E-09"
+        iyy="1.39449003709198E-06"
+        iyz="-1.56865788651068E-08"
+        izz="1.2847781945381E-05" />
+    </inertial>
+    <visual>
+      <origin
+        xyz="0 0 0"
+        rpy="0 0 0" />
+      <geometry>
+        <mesh
+          filename="file://$(find rosorin_description)/meshes/depth_camera_link.stl" />
+      </geometry>
+      <material
+        name="">
+        <color
+          rgba="0.792156862745098 0.819607843137255 0.933333333333333 1" />
+      </material>
+    </visual>
+    <collision>
+      <origin
+        xyz="0 0 0"
+        rpy="0 0 0" />
+      <geometry>
+        <mesh
+          filename="file://$(find rosorin_description)/meshes/depth_camera_link_collision.stl" />
+      </geometry>
+    </collision>
+  </link>
+  <joint
+    name="depth_camera"
+    type="fixed">
+    <origin
+      xyz="0.057373 7.9091E-05 0.091864"
+      rpy="0 0 0" />
+    <parent
+      link="base_link" />
+    <child
+      link="camera_link0" />
+    <axis
+      xyz="0 0 0" />
+  </joint>
+</robot>

File: install/rosorin_description/share/rosorin_description/urdf/dabai.xacro (robot description, xacro)
@@ -1 +1,57 @@
-/workspaces/ros2_ws/build/rosorin_description/urdf/dabai.xacro
+<?xml version="1.0" encoding="utf-8"?>
+<robot name="camera" xmlns:xacro="http://ros.org/wiki/xacro" >
+  <xacro:property name="M_PI"   value="3.1415926535897931"/>
+  <link
+    name="depth_cam_link">
+    <inertial>
+      <origin
+        xyz="0.00232981322860787 0.000387137406184821 -2.84059740606052E-05"
+        rpy="0 0 0" />
+      <mass
+        value="0.015428" />
+      <inertia
+        ixx="1.3945E-06"
+        ixy="-1.5684E-08"
+        ixz="-2.3104E-07"
+        iyy="1.2848E-05"
+        iyz="1.3156E-09"
+        izz="1.361E-05" />
+    </inertial>
+    <visual>
+      <origin
+        xyz="0 0 0"
+        rpy="0 0 0" />
+      <geometry>
+        <mesh
+          filename="file://$(find rosorin_description)/meshes/dabai_cam_link.STL" />
+      </geometry>
+      <material
+        name="">
+        <color
+          rgba="0.753 0.753 0.753 1" />
+      </material>
+    </visual>
+    <collision>
+      <origin
+        xyz="0 0 0"
+        rpy="0 0 0" />
+      <geometry>
+        <mesh
+          filename="file://$(find rosorin_description)/meshes/dabai_cam_link_collision.stl" />
+      </geometry>
+    </collision>
+  </link>
+  <joint
+    name="depth_cam_joint"
+    type="fixed">
+    <origin
+      xyz="0.057373 7.9091E-05 0.091864"
+      rpy="0 0 0" />
+    <parent
+      link="base_link" />
+    <child
+      link="depth_cam_link" />
+    <axis
+      xyz="0 0 0" />
+  </joint>
+</robot>

File: install/rosorin_description/share/rosorin_description/urdf/materials.xacro (robot description, xacro)
@@ -1 +1,27 @@
-/workspaces/ros2_ws/build/rosorin_description/urdf/materials.xacro
+<?xml version="1.0"?>
+<robot>
+    <material name="black">
+        <color rgba="0.3 0.3 0.3 1.0"/>
+    </material>
+    <material name="blue">
+        <color rgba="0.0 0.0 0.8 1.0"/>
+    </material>
+    <material name="green">
+        <color rgba="0.4 0.9 0.4 1.0"/>
+    </material>
+    <material name="gray">
+        <color rgba="0.7 0.7 0.7 1.0"/>
+    </material>
+    <material name="darkgray">
+        <color rgba="0.3 0.3 0.3 1.0"/>
+    </material>
+    <material name="red">
+        <color rgba="0.8 0.0 0.0 1.0"/>
+    </material>
+    <material name="white">
+        <color rgba="1.0 1.0 1.0 1.0"/>
+    </material>
+    <material name="yellow">
+        <color rgba="0.8 0.8 0.0 1.0"/>
+    </material>
+</robot>

File: install/rosorin_description/share/rosorin_description/urdf/rosorin.xacro (robot description, xacro)
@@ -1 +1,365 @@
-/workspaces/ros2_ws/build/rosorin_description/urdf/rosorin.xacro
+<?xml version="1.0" encoding="utf-8"?>
+<robot name="car" xmlns:xacro="http://ros.org/wiki/xacro" >
+  <xacro:property name="camera_type"    value="$(env DEPTH_CAMERA_TYPE)"/>
+  <xacro:include filename="$(find rosorin_description)/urdf/materials.xacro"/>
+  <link name="base_footprint"/>
+  <joint name="base_joint" type="fixed">
+    <parent link="base_footprint"/>
+    <child link="base_link"/>
+    <origin xyz="0.0 0.0 0.028" rpy="0 0 0"/>
+  </joint>
+  <link name="imu_link"/>
+  <joint name="imu_joint" type="fixed">
+    <parent link="base_link"/>
+    <child link="imu_link"/>
+    <origin xyz="0.04 -0.015 0.05" rpy="0 0 1.57"/>
+  </joint>
+  <link
+    name="base_link">
+    <inertial>
+      <origin
+        xyz="-0.0073743 0.00027245 0.033869"
+        rpy="0 0 0" />
+      <mass
+        value="0.05536" />
+      <inertia
+        ixx="0.00029526"
+        ixy="-8.622E-07"
+        ixz="3.753E-05"
+        iyy="0.00065872"
+        iyz="-4.6067E-09"
+        izz="0.00086726" />
+    </inertial>
+    <visual>
+      <origin
+        xyz="0 0 0"
+        rpy="0 0 0" />
+      <geometry>
+        <mesh
+          filename="file://$(find rosorin_description)/meshes/base_link.stl" />
+      </geometry>
+      <material
+        name="">
+        <color
+          rgba="0.5 0.5 0.5 1" />
+      </material>
+    </visual>
+    <collision>
+      <origin
+        xyz="0 0 0"
+        rpy="0 0 0" />
+      <geometry>
+        <mesh
+          filename="file://$(find rosorin_description)/meshes/base_link_collision.stl" />
+      </geometry>
+    </collision>
+  </link>
+  <link
+    name="lidar_frame">
+    <inertial>
+      <origin
+        xyz="8.95497003335615E-05 6.44963541535514E-05 -0.011400348556056"
+        rpy="0 0 0" />
+      <mass
+        value="0.0385600938526619" />
+      <inertia
+        ixx="4.66264138781846E-06"
+        ixy="-1.60730633906311E-07"
+        ixz="2.05163088641334E-09"
+        iyy="4.71595831823178E-06"
+        iyz="1.10063023333176E-08"
+        izz="7.61240253383846E-06" />
+    </inertial>
+    <visual>
+      <origin
+        xyz="0 0 0"
+        rpy="0 0 0" />
+      <geometry>
+        <mesh
+          filename="file://$(find rosorin_description)/meshes/lidar_link.stl" />
+      </geometry>
+      <material name="black"/>
+    </visual>
+    <collision>
+      <origin
+        xyz="0 0 0"
+        rpy="0 0 0" />
+      <geometry>
+        <mesh
+          filename="file://$(find rosorin_description)/meshes/lidar_link_collision.stl" />
+      </geometry>
+    </collision>
+  </link>
+  <joint
+    name="lidar"
+    type="fixed">
+    <origin
+      xyz="0.011476 7.415E-05 0.13641"
+      rpy="0 0 0" />
+    <parent
+      link="base_link" />
+    <child
+      link="lidar_frame" />
+    <axis
+      xyz="0 0 0" />
+  </joint>
+  <link
+    name="left_front_wheel_link">
+    <inertial>
+      <origin
+        xyz="6.78850066051367E-05 0.0194273902243469 4.2771032181671E-05"
+        rpy="0 0 0" />
+      <mass
+        value="0.0705101646075632" />
+      <inertia
+        ixx="1.05359955410655E-05"
+        ixy="-4.17160486096137E-09"
+        ixz="-3.48250757597355E-08"
+        iyy="1.65950885885739E-05"
+        iyz="4.89765791745149E-09"
+        izz="1.05450583464434E-05" />
+    </inertial>
+    <visual>
+      <origin
+        xyz="0 0 0"
+        rpy="0 0 0" />
+      <geometry>
+        <mesh
+          filename="file://$(find rosorin_description)/meshes/left_front_wheel_link.stl" />
+      </geometry>
+      <material name="black"/>
+    </visual>
+    <collision>
+      <origin
+        xyz="0 0 0"
+        rpy="0 0 0" />
+      <geometry>
+        <mesh
+          filename="file://$(find rosorin_description)/meshes/left_front_wheel_link_collision.stl" />
+      </geometry>
+    </collision>
+  </link>
+  <joint
+    name="left_front_wheel"
+    type="fixed">
+    <origin
+      xyz="0.09097 0.067865 0.017096"
+      rpy="0 0 0" />
+    <parent
+      link="base_link" />
+    <child
+      link="left_front_wheel_link" />
+    <axis
+      xyz="0 0 0" />
+  </joint>
+  <link
+    name="left_back_wheel_link">
+    <inertial>
+      <origin
+        xyz="-6.79935957126898E-05 0.0194272724865622 4.18919442857144E-05"
+        rpy="0 0 0" />
+      <mass
+        value="0.0705098315712721" />
+      <inertia
+        ixx="1.05363965532436E-05"
+        ixy="4.22186803055192E-09"
+        ixz="3.45056141524137E-08"
+        iyy="1.65964488067E-05"
+        iyz="4.90631628693761E-09"
+        izz="1.05458413899706E-05" />
+    </inertial>
+    <visual>
+      <origin
+        xyz="0 0 0"
+        rpy="0 0 0" />
+      <geometry>
+        <mesh
+          filename="file://$(find rosorin_description)/meshes/left_back_wheel_link.stl" />
+      </geometry>
+      <material name="black"/>
+    </visual>
+    <collision>
+      <origin
+        xyz="0 0 0"
+        rpy="0 0 0" />
+      <geometry>
+        <mesh
+          filename="file://$(find rosorin_description)/meshes/left_back_wheel_link_collision.stl" />
+      </geometry>
+    </collision>
+  </link>
+  <joint
+    name="left_back_wheel"
+    type="fixed">
+    <origin
+      xyz="-0.080677 0.067865 0.016719"
+      rpy="0 0 0" />
+    <parent
+      link="base_link" />
+    <child
+      link="left_back_wheel_link" />
+    <axis
+      xyz="0 0 0" />
+  </joint>
+  <link
+    name="right_front_wheel_link">
+    <inertial>
+      <origin
+        xyz="6.56410494759008E-05 -0.0194272432930035 4.09111593353481E-05"
+        rpy="0 0 0" />
+      <mass
+        value="0.0705098464929629" />
+      <inertia
+        ixx="1.0536754444795E-05"
+        ixy="4.2338086716559E-09"
+        ixz="-3.43871505647673E-08"
+        iyy="1.6596872052673E-05"
+        iyz="-4.91902435337096E-09"
+        izz="1.05459220480947E-05" />
+    </inertial>
+    <visual>
+      <origin
+        xyz="0 0 0"
+        rpy="0 0 0" />
+      <geometry>
+        <mesh
+          filename="file://$(find rosorin_description)/meshes/right_front_wheel_link.stl" />
+      </geometry>
+      <material name="black"/>
+    </visual>
+    <collision>
+      <origin
+        xyz="0 0 0"
+        rpy="0 0 0" />
+      <geometry>
+        <mesh
+          filename="file://$(find rosorin_description)/meshes/right_front_wheel_link_collision.stl" />
+      </geometry>
+    </collision>
+  </link>
+  <joint
+    name="right_front_wheel"
+    type="fixed">
+    <origin
+      xyz="0.090972 -0.067717 0.017098"
+      rpy="0 0 0" />
+    <parent
+      link="base_link" />
+    <child
+      link="right_front_wheel_link" />
+    <axis
+      xyz="0 0 0" />
+  </joint>
+  <link
+    name="right_back_wheel_link">
+    <inertial>
+      <origin
+        xyz="-4.8854E-05 -0.017043 1.8927E-05"
+        rpy="0 0 0" />
+      <mass
+        value="0.058672" />
+      <inertia
+        ixx="6.7699E-06"
+        ixy="-1.99E-08"
+        ixz="1.4456E-08"
+        iyy="9.6881E-06"
+        iyz="1.0739E-08"
+        izz="6.7781E-06" />
+    </inertial>
+    <visual>
+      <origin
+        xyz="0 0 0"
+        rpy="0 0 0" />
+      <geometry>
+        <mesh
+          filename="file://$(find rosorin_description)/meshes/right_back_wheel_link.stl" />
+      </geometry>
+      <material name="black"/>
+    </visual>
+    <collision>
+      <origin
+        xyz="0 0 0"
+        rpy="0 0 0" />
+      <geometry>
+        <mesh
+          filename="file://$(find rosorin_description)/meshes/right_back_wheel_link_collision.stl" />
+      </geometry>
+    </collision>
+  </link>
+  <joint
+    name="right_back_wheel"
+    type="fixed">
+    <origin
+      xyz="-0.080677 -0.067717 0.016719"
+      rpy="0 0 0" />
+    <parent
+      link="base_link" />
+    <child
+      link="right_back_wheel_link" />
+    <axis
+      xyz="0 0 0" />
+  </joint>
+  <link
+    name="mic_link">
+    <inertial>
+      <origin
+        xyz="-7.65493159082808E-07 -0.0249662719365599 0.0134328993494675"
+        rpy="0 0 0" />
+      <mass
+        value="0.0210934941268813" />
+      <inertia
+        ixx="1.36191114404946E-05"
+        ixy="-4.3417522172067E-10"
+        ixz="-1.27861440031619E-10"
+        iyy="3.01739703567571E-05"
+        iyz="4.99987016844085E-11"
+        izz="4.19372593423754E-05" />
+    </inertial>
+    <visual>
+      <origin
+        xyz="0 0 0"
+        rpy="0 0 0" />
+      <geometry>
+        <mesh
+          filename="file://$(find rosorin_description)/meshes/mic_link.stl" />
+      </geometry>
+      <material name="black"/>
+    </visual>
+    <collision>
+      <origin
+        xyz="0 0 0"
+        rpy="0 0 0" />
+      <geometry>
+        <mesh
+          filename="file://$(find rosorin_description)/meshes/mic_link_collision.stl" />
+      </geometry>
+    </collision>
+  </link>
+  <joint
+    name="mic"
+    type="fixed">
+    <origin
+      xyz="-0.068965 0.025075 0.10955"
+      rpy="0 0 0" />
+    <parent
+      link="base_link" />
+    <child
+      link="mic_link" />
+    <axis
+      xyz="0 0 0" />
+  </joint>
+  <link name="lidar_sim_frame" />
+  <joint
+    name="lidar_sim_frame_joint"
+    type="fixed">
+    <origin xyz="0 0 0" rpy="0 0 0" />
+    <parent link="lidar_frame" />
+    <child link="lidar_sim_frame" />
+  </joint>
+  <xacro:if value="${camera_type == 'AsCamera' or camera_type == 'aurora'}">
+    <xacro:include filename="$(find rosorin_description)/urdf/ascamera.xacro"/>
+  </xacro:if>
+  <xacro:if value="${camera_type == 'Dabai'}">
+    <xacro:include filename="$(find rosorin_description)/urdf/dabai.xacro"/>
+  </xacro:if>
+</robot>
